Commit message: Updated urdf of workcell to include glass walls in workcell

File: fanuc_lrmate200ic_support/urdf/intern_demo_workcell.xacro (robot description, xacro)
@@ -6,5 +6,5 @@
   <!-- Add World -->
   <material name="light_gray">
-    <color rgba="0.7 0.7 0.7 1"/>
+    <color rgba="0.7 0.7 0.7 0.5"/>
   </material>
   <material name="dark_gray">
@@ -38,4 +38,73 @@
     <child link="floor"/>
   </joint>
+    <!-- Add Walls for Collision -->
+    <xacro:property name="lengthw" value="1.171575"/>
+    <xacro:property name="widthw" value="1.11125"/>
+    <!-- Right Wall -->
+    <link name="wall_right">
+      <visual>
+        <origin xyz="0.0508 -${width/2+0.01905} ${0.001+widthw/2}" rpy="${pi/2} 0 0"/>
+        <geometry>
+          <box size="${lengthw-0.0508} ${widthw} 0.001"/>
+        </geometry>
+        <material name="light_gray"/>
+      </visual>
+      <collision>
+        <origin xyz="0.0508 -${width/2+0.01905} ${0.001+widthw/2}" rpy="${pi/2} 0 0"/>
+        <geometry>
+          <box size="${lengthw-0.0508} ${widthw} 0.001"/>
+        </geometry>
+        <material name="light_gray"/>
+      </collision>
+    </link>
+    <joint name="floor_to_wall_right" type="fixed">
+      <origin xyz="0 0 0" rpy="0 0 0"/>
+      <parent link="floor"/>
+      <child link="wall_right"/>
+    </joint>
+    <!-- Back Wall -->
+    <link name="wall_back">
+      <visual>
+        <origin xyz="${length/2+0.009525} 0 ${0.001+widthw/2}" rpy="${pi/2} 0 ${pi/2}"/>
+        <geometry>
+          <box size="${width} ${widthw} 0.001"/>
+        </geometry>
+        <material name="light_gray"/>
+      </visual>
+      <collision>
+        <origin xyz="${length/2+0.009525} 0 ${0.001+widthw/2}" rpy="${pi/2} 0 ${pi/2}"/>
+        <geometry>
+          <box size="${width} ${widthw} 0.001"/>
+        </geometry>
+        <material name="light_gray"/>
+      </collision>
+    </link>
+    <joint name="floor_to_wall_back" type="fixed">
+      <origin xyz="0 0 0" rpy="0 0 0"/>
+      <parent link="floor"/>
+      <child link="wall_back"/>
+    </joint>
+    <!-- Front Wall -->
+    <link name="wall_front">
+      <visual>
+        <origin xyz="-${length/2-0.0762} 0 ${0.001+widthw/2}" rpy="${pi/2} 0 ${pi/2}"/>
+        <geometry>
+          <box size="${width} ${widthw} 0.001"/>
+        </geometry>
+        <material name="light_gray"/>
+      </visual>
+      <collision>
+      <origin xyz="-${length/2-0.0762} 0 ${0.001+widthw/2}" rpy="${pi/2} 0 ${pi/2}"/>
+        <geometry>
+          <box size="${width} ${widthw} 0.001"/>
+        </geometry>
+        <material name="light_gray"/>
+      </collision>
+    </link>
+    <joint name="floor_to_wall_front" type="fixed">
+      <origin xyz="0 0 0" rpy="0 0 0"/>
+      <parent link="floor"/>
+      <child link="wall_front"/>
+    </joint>
   <!-- Add Acryllic-->
     <xacro:property name="lengtha" value="0.923925"/>
@@ -44,5 +113,5 @@
     <link name="acryllic">
       <visual>
-        <origin xyz="${0.14605} -${0.0254} ${0.001+thicknessa_plus_p/2}"/>
+        <origin xyz="0 0 ${0.001+thicknessa_plus_p/2}"/>
         <geometry>
           <box size="${lengtha} ${widtha} ${thicknessa_plus_p}"/>
@@ -65,7 +134,7 @@
   <link name="ceiling">
     <visual>
-      <origin xyz="0 -${0/10} 0.001" rpy="0 0 0"/>
-      <geometry>
-        <box size="${length} ${width} 0.001"/>
+      <origin xyz="0.0508 -${0/10} 0.001" rpy="0 0 0"/>
+      <geometry>3.3125+7.375/2
+        <box size="${length-0.0508} ${width} 0.001"/>
       </geometry>
     </visual>
@@ -85,5 +154,5 @@
     <parent link="ceiling"/>
     <child link="base_link"/>
-    <origin xyz="-0.3737705 -0.169135 0" rpy="0 -3.14 -3.14"/>
+    <origin xyz="-${length/2-2*0.0508-0.1778} -0.169135 0" rpy="0 -3.14 -3.14"/>
   </joint>
   <!-- Create a frame representing the robot tool flange (behind the teach tool and nominal tool0 frame) for IKFast -->

Commit message: Updated collision matrix for moveit and updated colors for urdf

File: fanuc_lrmate200ic_support/urdf/intern_demo_workcell.xacro (robot description, xacro)
@@ -14,4 +14,7 @@
     <color rgba="0 0 1 1"/>
   </material>
+  <material name="black">
+    <color rgba="0 0 0 1"/>
+  </material>
   <link name="world"/>
   <!-- Add Floor -->
@@ -55,5 +58,4 @@
           <box size="${lengthw-0.0508} ${widthw} 0.001"/>
         </geometry>
-        <material name="light_gray"/>
       </collision>
     </link>
@@ -77,5 +79,4 @@
           <box size="${width} ${widthw} 0.001"/>
         </geometry>
-        <material name="light_gray"/>
       </collision>
     </link>
@@ -99,5 +100,4 @@
           <box size="${width} ${widthw} 0.001"/>
         </geometry>
-        <material name="light_gray"/>
       </collision>
     </link>
@@ -109,5 +109,5 @@
   <!-- Add Acryllic-->
     <xacro:property name="lengtha" value="0.923925"/>
-    <xacro:property name="widtha" value="0.8763"/>
+    <xacro:property name="widtha" value="0.8763"/>black
     <xacro:property name="thicknessa_plus_p" value="${0.01+0.0047625}"/>
     <link name="acryllic">
@@ -138,4 +138,5 @@
         <box size="${length-0.0508} ${width} 0.001"/>
       </geometry>
+      <material name="black"/>
     </visual>
     <collision>
@@ -172,4 +173,5 @@
         <cylinder length="${ee_length}" radius="${ee_radius}"/>
       </geometry>
+      <material name="black"/>
     </visual>
     <collision>
